Commit message: Retuned the controllers

File: ros1/ball_chaser_ws/src/my_robot/urdf/my_robot.urdf (robot description, URDF)
Before this commit: robot my_robot, 7 links, 6 joints
Links:
- removed link back_left_wheel
- removed link back_right_wheel
- removed link camera_link
- removed link front_left_wheel
- removed link front_right_wheel
- removed link lidar_link
- added link left_wheel, mass 2; collision sphere radius=0.3; visual sphere radius=0.3
- added link right_wheel, mass 2; collision sphere radius=0.3; visual sphere radius=0.3
- link base_link: mass 144.435621199277 -> 1.14395; geometry collision box size=2.01142 1 0.568726; visual box size=2.01142 1 0.568726
Joints:
- removed joint back_left_wheel_joint
- removed joint back_right_wheel_joint
- removed joint camera_link_joint
- removed joint front_left_wheel_joint
- removed joint front_right_wheel_joint
- removed joint lidar_link_joint
- added joint left_wheel_joint: type revolute, parent base_link, child left_wheel, origin xyz=0.554283 0.625029 -0.025 rpy= 0 -0 0, axis 0 0 1, limit lower=-1.79769e+308 upper=1.79769e+308 effort=-1 velocity=-1
- added joint right_wheel_joint: type revolute, parent base_link, child right_wheel, origin xyz=0.554282 -0.625029 -0.025 rpy= 0 -0 0, axis 0 0 1, limit lower=-1.79769e+308 upper=1.79769e+308 effort=-1 velocity=-1

Commit message: Update to skid drive robot

File: ros1/ball_chaser_ws/src/my_robot/urdf/my_robot.urdf (robot description, URDF)
Before this commit: robot my_robot, 3 links, 2 joints
Links:
- removed link left_wheel
- removed link right_wheel
- added link back_left_wheel, mass 10.426; collision mesh filename=package://my_robot/meshes/back_left_wheel.STL; visual mesh filename=package://my_robot/meshes/back_left_wheel.STL
- added link back_right_wheel, mass 10.426; collision mesh filename=package://my_robot/meshes/back_right_wheel.STL; visual mesh filename=package://my_robot/meshes/back_right_wheel.STL
- added link camera_link, mass 0.016141; collision mesh filename=package://my_robot/meshes/camera_link.STL; visual mesh filename=package://my_robot/meshes/camera_link.STL
- added link front_left_wheel, mass 10.426; collision mesh filename=package://my_robot/meshes/front_left_wheel.STL; visual mesh filename=package://my_robot/meshes/front_left_wheel.STL
- added link front_right_wheel, mass 10.426; collision mesh filename=package://my_robot/meshes/front_right_wheel.STL; visual mesh filename=package://my_robot/meshes/front_right_wheel.STL
- added link lidar_link, mass 0.016141; collision mesh filename=package://my_robot/meshes/lidar_link.STL; visual mesh filename=package://my_robot/meshes/lidar_link.STL
- link base_link: mass 1.14395 -> 144.435621199277; geometry collision mesh filename=package://my_robot/meshes/base_link.STL; visual mesh filename=package://my_robot/meshes/base_link.STL
Joints:
- removed joint left_wheel_joint
- removed joint right_wheel_joint
- added joint back_left_wheel_joint: type continuous, parent base_link, child back_left_wheel, origin xyz=-0.82 0.34 -0.031041 rpy=0 0 0, axis 0 1 0
- added joint back_right_wheel_joint: type continuous, parent base_link, child back_right_wheel, origin xyz=-0.82 -0.3358 -0.031041 rpy=0 0 0, axis 0 1 0
- added joint camera_link_joint: type fixed, parent lidar_link, child camera_link, origin xyz=0 0 0.01 rpy=0 0 0, axis 0 0 0
- added joint front_left_wheel_joint: type continuous, parent base_link, child front_left_wheel, origin xyz=0.2176 0.34 -0.031041 rpy=0 0 0, axis 0 1 0
- added joint front_right_wheel_joint: type continuous, parent base_link, child front_right_wheel, origin xyz=0.2176 -0.3358 -0.031041 rpy=0 0 0, axis 0 1 0
- added joint lidar_link_joint: type fixed, parent base_link, child lidar_link, origin xyz=0.15965 0.0021 0.1103 rpy=0 0 0, axis 0 0 0
